File: SmartEffector/SmartEffector_v2.0/SmartEffector.sch (KiCad schematic (older format))
At the start: 57 parts, among them M1 FID, M10 M_2.9mm, M11 M_2.9mm, M13 Ziptie, M16 12mm, M2 FID, M3 M_2.9mm, M4 M_2.9mm, M5 M_2.9mm, M6 M_2.9mm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

Commit message: Updated some schematic issues
Parts:
- added M15: Duet3D Logo, complib:LOGO_Duet3dCompatible, symbol Duet3:Duet3D_Logo
- C6: value 22u<20% -> 22u
- M1, M2: symbol smart:FID -> Mechanical:Fiducial
- M10, M11, M13, M3, M4, M5, M6, M7, M8, M9: symbol Mechanical:Mounting_Hole -> Mechanical:MountingHole
- M16: symbol smart:FID -> Mechanical:MountingHole
- U1: symbol smart:LDK130M08 -> Regulator_Linear:LDK130-10_SOT23_SOT353
- U2: value ATtiny44A-MMH-PAD -> ATtiny44A-MUR; symbol MCU_Microchip_ATtiny:ATtiny44A-MMH-PAD -> SmartEffector-rescue:ATtiny44A-MMH-PAD-MCU_Microchip_ATtiny
- U3: symbol smart:MCP6286 -> Amplifier_Operational:MCP6286
Changed lines of the file:
@@
 EESchema Schematic File Version 4
 LIBS:SmartEffector-cache
-EELAYER 26 0
+EELAYER 30 0
 EELAYER END
 $Descr A4 11693 8268
@@
 $EndComp
 $Comp
-L Mechanical:Mounting_Hole M4
+L Mechanical:MountingHole M4
 U 1 1 587CEA49
 P 1660 7005
@@
 $EndComp
 $Comp
-L Mechanical:Mounting_Hole M5
+L Mechanical:MountingHole M5
 U 1 1 587CF0CA
 P 2160 7005
@@
 $EndComp
 $Comp
-L Mechanical:Mounting_Hole M6
+L Mechanical:MountingHole M6
 U 1 1 587CF116
 P 2610 7005
@@
 $EndComp
 $Comp
-L Mechanical:Mounting_Hole M7
+L Mechanical:MountingHole M7
 U 1 1 587CF163
 P 3060 7005
@@
 $EndComp
 $Comp
-L Mechanical:Mounting_Hole M8
+L Mechanical:MountingHole M8
 U 1 1 587CF1AF
 P 3510 7005
@@
 $EndComp
 $Comp
-L Mechanical:Mounting_Hole M3
+L Mechanical:MountingHole M3
 U 1 1 587CF200
 P 1210 7005
@@
 $EndComp
 $Comp
-L smart:FID M1
+L Mechanical:Fiducial M1
 U 1 1 587CF312
 P 1400 7515
@@
 $EndComp
 $Comp
-L smart:FID M2
+L Mechanical:Fiducial M2
 U 1 1 587CF390
 P 1650 7515
@@
 Heater and Fan\npass through
 $Comp
-L Mechanical:Mounting_Hole M13
+L Mechanical:MountingHole M13
 U 1 1 587E7263
 P 3010 7505
@@
 $EndComp
 $Comp
+L Duet3:Duet3D_Logo M15
+U 1 1 587ED2EE
+P 810 7485
+F 0 "M15" H 810 7335 60  0000 C CNN
+F 1 "Duet3D Logo" H 810 7635 60  0000 C CNN
+F 2 "complib:LOGO_Duet3dCompatible" H 810 7485 60  0001 C CNN
+F 3 "" H 810 7485 60  0000 C CNN
+	1    810  7485
+	1    0    0    -1
+$EndComp
+$Comp
 L Device:LED_Small D1
 U 1 1 58800164
@@
 T
 $Comp
-L smart:FID M16
+L Mechanical:MountingHole M16
 U 1 1 5897DC47
 P 2050 7515
@@
 $EndComp
 $Comp
-L smart:MCP6286 U3
+L Amplifier_Operational:MCP6286 U3
 U 1 1 58D2A7FE
 P 8550 1775
@@
 P 8670 2425
 F 0 "C6" V 8770 2425 50  0000 L CNN
-F 1 "22u<20%" V 8560 2245 50  0000 L CNN
+F 1 "22u" V 8560 2245 50  0000 L CNN
 F 2 "complib:C_0805" H 8670 2425 50  0001 C CNN
 F 3 "" H 8670 2425 50  0000 C CNN
@@
 Connection ~ 1950 3225
 $Comp
-L Mechanical:Mounting_Hole M11
-U 1 1 59524255
-P 2380 6425
-F 0 "M11" H 2380 6275 60  0000 C CNN
-F 1 "M_2.9mm" H 2380 6575 60  0000 C CNN
-F 2 "complib:MountingHole_2.9mm" H 2380 6425 60  0001 C CNN
-F 3 "" H 2380 6425 60  0000 C CNN
-	1    2380 6425
-	1    0    0    -1
-$EndComp
-$Comp
-L Mechanical:Mounting_Hole M9
+L Mechanical:MountingHole M9
 U 1 1 59524330
 P 2870 6415
@@
 $EndComp
 $Comp
-L Mechanical:Mounting_Hole M10
+L Mechanical:MountingHole M10
 U 1 1 595243F8
 P 3370 6415
@@
 	1950 3225 2900 3225
 $Comp
-L MCU_Microchip_ATtiny:ATtiny44A-MMH-PAD U2
+L SmartEffector-rescue:ATtiny44A-MMH-PAD-MCU_Microchip_ATtiny U2
 U 1 1 5BC6AD32
 P 9050 3775
 F 0 "U2" H 8171 3821 50  0000 R CNN
-F 1 "ATtiny44A-MMH-PAD" H 9425 3750 50  0000 R CNN
+F 1 "ATtiny44A-MUR" H 9425 3750 50  0000 R CNN
 F 2 "complib:QFN-20-1EP_4x4mm_Pitch0.5mm" H 9050 3775 50  0001 C CIN
 F 3 "" H 9050 3775 50  0001 C CNN
@@
 	6600 1650 6600 1475
 Connection ~ 6600 1650
-Wire Wire Line
-	5425 1250 4875 1250
 Connection ~ 5425 1250
 Wire Wire Line
-	4925 1625 4925 1550
-Wire Wire Line
-	4925 1550 4875 1550
-Wire Wire Line
 	4925 1825 4925 1925
 Wire Wire Line
@@
 	4400 1925 4400 1950
 Wire Wire Line
-	4400 1925 4400 1400
-Wire Wire Line
-	4400 1400 3875 1400
-Connection ~ 4400 1925
-Wire Wire Line
-	3875 1550 3825 1550
-Wire Wire Line
-	3825 1550 3825 1250
-Wire Wire Line
-	3875 1250 3825 1250
-Wire Wire Line
-	3825 1250 3825 775
-Wire Wire Line
 	3825 775  9050 775
-Connection ~ 3825 1250
 Wire Wire Line
 	9050 775  9050 885
 $Comp
-L smart:LDK130M08 U1
+L Regulator_Linear:LDK130-10_SOT23_SOT353 U1
 U 1 1 58D58578
-P 4375 1400
-F 0 "U1" H 4375 1550 60  0000 C CNN
-F 1 "LDK130M10" H 4360 1735 60  0000 C CNN
-F 2 "complib:SOT-23-5L" H 4375 1400 60  0001 C CNN
-F 3 "" H 4375 1400 60  0000 C CNN
-	1    4375 1400
+P 4375 1350
+F 0 "U1" H 4375 1500 60  0000 C CNN
+F 1 "LDK130M10" H 4360 1685 60  0000 C CNN
+F 2 "complib:SOT-23-5L" H 4375 1350 60  0001 C CNN
+F 3 "" H 4375 1350 60  0000 C CNN
+	1    4375 1350
 	1    0    0    -1
 $EndComp
@@
 Wire Wire Line
 	10725 6075 10600 6075
+$Comp
+L Mechanical:MountingHole M11
+U 1 1 59524255
+P 2380 6425
+F 0 "M11" H 2380 6275 60  0000 C CNN
+F 1 "M_2.9mm" H 2380 6575 60  0000 C CNN
+F 2 "complib:MountingHole_2.9mm" H 2380 6425 60  0001 C CNN
+F 3 "" H 2380 6425 60  0000 C CNN
+	1    2380 6425
+	1    0    0    -1
+$EndComp
+Wire Wire Line
+	4400 1925 4375 1925
+Wire Wire Line
+	4375 1925 4375 1650
+Connection ~ 4400 1925
+Wire Wire Line
+	4075 1350 3825 1350
+Wire Wire Line
+	3825 775  3825 1250
+Wire Wire Line
+	4075 1250 3825 1250
+Connection ~ 3825 1250
+Wire Wire Line
+	3825 1250 3825 1350
+Wire Wire Line
+	4925 1350 4675 1350
+Wire Wire Line
+	4925 1350 4925 1625
+Wire Wire Line
+	4675 1250 5425 1250
 $EndSCHEMATC
